File: light sensor basic.brd (EAGLE design)
At the start: 83.2 x 57.8 mm, 1 part

Commit message: Eagle 2
Eagle 2
Parts:
- added C1: (no value), rcl:C1206
- added J1: UJ2-MIBH-G-SMT-TR, UJ2-MIBH-G-SMT-TR:CUI_UJ2-MIBH-G-SMT-TR
- added LED1: (no value), led:SML0805
- added R1, TP1, TP2, TP3, TP4: (no value), rcl:R1206
- added R2: TC33X-2-203E, TC33X-2-203E:TRIM_TC33X-2-203E
- added R3: 150, rcl:R0805
- added T1: (no value), transistor:SOT23-EBC
- added U1: VCNT2020, VCNT2020:XDCR_VCNT2020
- moved U$1 106.9 mm to (-106.7, 6.35)
Connections:
- new net GND: C1.1, J1.5, J1.S1, J1.S2, J1.S3, J1.S4, R2.3, T1.E, TP4.1, TP4.2, U1.4
- new net N$1: R1.2, U1.3
- new net N$3: R2.2, T1.B, TP2.1, TP2.2
- new net N$4: LED1.A, R3.1
- new net N$5: LED1.C, T1.C
- new net TP1: R2.1, TP1.1, TP1.2, U1.1
- new net VCC: C1.2, J1.1, R1.1, R3.2, TP3.1, TP3.2, U1.2
Routing:
- net GND: track 0.00 -> 63.9 mm
- net VCC: track 0.00 -> 62.5 mm
- net TP1: track 0.00 -> 55.3 mm
- net N$3: track 0.00 -> 21.6 mm
- net N$1: track 0.00 -> 7.22 mm
- net N$4: track 0.00 -> 6.89 mm
- net N$5: track 0.00 -> 4.20 mm
- added copper zone on layer 1, net N$2
Other:
- board size 83.2 x 57.8 mm -> 160 x 100 mm
- board text added: "C1"
- board text added: "K<- LED1"
- board text added: "R1"
- board text added: "R2"
- board text added: "R3"
- board text added: "T1"
- board text added: "TP1"
- board text added: "TP2"
- board text added: "TP3"
- board text added: "TP4"
- board text added: "U1"
